File: project/esp32c5-airunit-nano.kicad_pcb (KiCad board)
At the start: 2 copper layers, 19.7 x 22.9 mm, 2 parts, among them J1 Conn_01x24_MountingPin, U1 ESP32-C5-WROOM-1U

Commit message: i've updated the project files
! ! ! STILL UNFINISHED ! ! !
Parts:
- added C1: 10uF, Capacitor_SMD:C_0603_1608Metric, F.Cu at (153.4, 72.4)
- added C10: 10uF, Capacitor_SMD:C_0603_1608Metric, F.Cu at (153.8, 83.5)
- added C11: 10uF, Capacitor_SMD:C_0603_1608Metric, F.Cu at (147.6, 83.5)
- added C12: 100nF, Capacitor_SMD:C_0603_1608Metric, F.Cu at (156.6, 73.3)
- added C13: 10uF, Capacitor_SMD:C_0603_1608Metric, F.Cu at (156.7, 71.5)
- added C2: 10uF, Capacitor_SMD:C_0603_1608Metric, F.Cu at (156.4, 77.2)
- added C3: 100nF, Capacitor_SMD:C_0603_1608Metric, F.Cu at (156.4, 78.7)
- added C4: 10uF, Capacitor_SMD:C_0603_1608Metric, F.Cu at (152.6, 79.3)
- added C5: 10uF, Capacitor_SMD:C_0603_1608Metric, F.Cu at (148.3, 76.4)
- added C6: 10uF, Capacitor_SMD:C_0603_1608Metric, F.Cu at (148.4, 72.3)
- added C7: 10uF, Capacitor_SMD:C_0603_1608Metric, F.Cu at (153.4, 76.4)
- added C8: 10uF, Capacitor_SMD:C_0603_1608Metric, F.Cu at (156.8, 83.5)
- added C9: 10uF, Capacitor_SMD:C_0603_1608Metric, F.Cu at (150.7, 83.5)
- added J3: Conn_02x03_Counter_Clockwise, Connector_PinSocket_1.27mm:PinSocket_2x03_P1.27mm_Vertical, F.Cu at (144.3, 80.6)
- added L1: FHD252012S-100MT, Inductor_SMD:L_Changjiang_FNR252010S, F.Cu at (152.6, 81.3)
- added U2: HX1001-GEC, Package_TO_SOT_SMD:TSOT-23-5, F.Cu at (156.4, 81.1)
- added U3: JTD6206-28, Package_TO_SOT_SMD:SOT-23, F.Cu at (150.9, 72.3)
- added U4: JTD6206-18, Package_TO_SOT_SMD:SOT-23, F.Cu at (150.9, 76.4)
- moved J1 0.34 mm to (149.3, 89.6)
Connections:
- J1 pad 1: unconnected-(J1-Pin_1-Pad1) -> +2V8
- J1 pad 10: unconnected-(J1-Pin_10-Pad10) -> GND
- J1 pad 11: unconnected-(J1-Pin_11-Pad11) -> y8
- J1 pad 12: unconnected-(J1-Pin_12-Pad12) -> xclk
- J1 pad 13: unconnected-(J1-Pin_13-Pad13) -> y9
- J1 pad 14: unconnected-(J1-Pin_14-Pad14) -> +1V8
- J1 pad 15: unconnected-(J1-Pin_15-Pad15) -> Net-(J1-Pin_15)
- J1 pad 2: unconnected-(J1-Pin_2-Pad2) -> GND
- J1 pad 20: unconnected-(J1-Pin_20-Pad20) -> scl
- J1 pad 21: unconnected-(J1-Pin_21-Pad21) -> +2V8
- J1 pad 22: unconnected-(J1-Pin_22-Pad22) -> sda
- J1 pad 23: unconnected-(J1-Pin_23-Pad23) -> GND
- J1 pad 3: unconnected-(J1-Pin_3-Pad3) -> y4
- J1 pad 4: unconnected-(J1-Pin_4-Pad4) -> y3
- J1 pad 5: unconnected-(J1-Pin_5-Pad5) -> y5
- J1 pad 6: unconnected-(J1-Pin_6-Pad6) -> y2
- J1 pad 7: unconnected-(J1-Pin_7-Pad7) -> y6
- J1 pad 8: unconnected-(J1-Pin_8-Pad8) -> pclk
- J1 pad 9: unconnected-(J1-Pin_9-Pad9) -> y7
- J1 pad MP: unconnected-(J1-MountPin-PadMP) -> GND
- U1 pad 1: Net-(U1-GND-Pad1) -> GND
- U1 pad 10: unconnected-(U1-GPIO8-Pad10) -> y4
- U1 pad 11: unconnected-(U1-GPIO9-Pad11) -> y3
- U1 pad 12: unconnected-(U1-GPIO10-Pad12) -> y2
- U1 pad 13: unconnected-(U1-GPIO13/USB_D--Pad13) -> usb_dn
- U1 pad 14: unconnected-(U1-GPIO14/USB_D+-Pad14) -> usb_dp
- U1 pad 18: unconnected-(U1-GPIO27-Pad18) -> uart2_tx
- U1 pad 2: unconnected-(U1-3V3-Pad2) -> +3V3
- U1 pad 24: unconnected-(U1-U0RXD/GPIO12-Pad24) -> uart0_rx
- U1 pad 25: unconnected-(U1-U0TXD/GPIO11-Pad25) -> uart0_tx
- U1 pad 26: unconnected-(U1-GPIO25-Pad26) -> scl
- U1 pad 27: unconnected-(U1-GPIO26-Pad27) -> sda
- U1 pad 28: Net-(U1-GND-Pad1) -> GND
- U1 pad 29: Net-(U1-GND-Pad1) -> GND
- U1 pad 3: unconnected-(U1-EN/CHIP_PU-Pad3) -> mcu_rst
- U1 pad 30: Net-(U1-GND-Pad1) -> GND
- U1 pad 32: Net-(U1-GND-Pad1) -> GND
- U1 pad 4: unconnected-(U1-GPIO2-Pad4) -> pclk
- U1 pad 5: unconnected-(U1-GPIO3-Pad5) -> y9
- U1 pad 6: unconnected-(U1-GPIO0-Pad6) -> y8
- U1 pad 7: unconnected-(U1-GPIO1-Pad7) -> y7
- U1 pad 8: unconnected-(U1-GPIO6-Pad8) -> y6
- U1 pad 9: unconnected-(U1-GPIO7-Pad9) -> y5

Commit message: i've updated the project files
we're actually getting somewhere, the layout is pretty close to what i would call not bad
Parts:
- removed C10, C11, C13, C9: 10uF, Capacitor_SMD:C_0603_1608Metric
- removed C12: 100nF, Capacitor_SMD:C_0603_1608Metric
- removed J3: Conn_02x03_Counter_Clockwise, Connector_PinSocket_1.27mm:PinSocket_2x03_P1.27mm_Vertical
- removed U3: JTD6206-28, Package_TO_SOT_SMD:SOT-23
- removed U4: JTD6206-18, Package_TO_SOT_SMD:SOT-23
- added D1: red, LED_SMD:LED_0603_1608Metric, F.Cu at (156.9, 71.2)
- added J2: Conn_01x01_Pin, Library:SolderWirePad_1x01_SMD_2x3mm, F.Cu at (141.7, 75.3)
- added J4: Conn_01x01_Pin, Library:SolderWirePad_1x01_SMD_2x3mm, F.Cu at (141.7, 78.4)
- added J5: Conn_01x01_Pin, Library:SolderWirePad_1x01_SMD_2x3mm, F.Cu at (157.1, 81.6)
- added J6: Conn_01x01_Pin, Library:SolderWirePad_1x01_SMD_2x3mm, F.Cu at (157.1, 78.4)
- added J7: Conn_01x01_Pin, Library:SolderWirePad_1x01_SMD_2x3mm, F.Cu at (157.1, 75.3)
- added J8: 0475710001, 0475710001:MOLEX_0475710001, F.Cu at (149.5, 79.9)
- added R1: 100kR, Resistor_SMD:R_0603_1608Metric, F.Cu at (151.2, 75.4)
- added R2: tbd, Resistor_SMD:R_0603_1608Metric, F.Cu at (149.6, 75.4)
- added R3: 220R, Resistor_SMD:R_0603_1608Metric, F.Cu at (156.9, 72.9)
- added R6: 100kR, Resistor_SMD:R_0603_1608Metric, F.Cu at (142.4, 81.4)
- added SW1: SW_Push, Button_Switch_SMD:SW_SPST_B3U-3000P-B, F.Cu at (142.5, 71.8)
- added Y1: YD24MUBCE2O, Oscillator:Oscillator_SMD_ECS_2520MV-xxx-xx-4Pin_2.5x2.0mm, F.Cu at (145.5, 75.4)
- C6: value 10uF -> 100nF
- J1: value Conn_01x24_MountingPin -> FPC0.5B-WTX-24P; footprint Connector_FFC-FPC:Hirose_FH12-24S-0.5SH_1x24-1MP_P0.50mm_Horizontal -> Connector_FFC-FPC:TE_2-1734839-4_1x24-1MP_P0.5mm_Horizontal
- L1: value FHD252012S-100MT -> FHD252010S-100MT
- U1: renamed from U2; value HX1001-GEC -> MT3406
- moved C5 17.3 mm to (157.0, 91.4), turned to 0 degrees
- moved C4 16.3 mm to (141.8, 91.4)
- moved C8 16.1 mm to (140.8, 81.4), turned to 90 degrees
- moved C1 12.2 mm to (146.0, 72.2), turned to -90 degrees
- moved U1 10.8 mm to (150.3, 72.2), turned to 0 degrees
- moved C2 10.2 mm to (147.5, 72.2), turned to -90 degrees
- moved L1 9.29 mm to (153.8, 72.1), turned to -90 degrees
- moved C6 6.63 mm to (154.3, 75.4)
- moved C7 5.49 mm to (148.0, 75.4)
- moved C3 3.09 mm to (152.7, 75.4), turned to -90 degrees
- moved J1 0.16 mm to (149.4, 89.5)
- moved U2 0.16 mm to (149.6, 81.5)
- renumbered C3 to C1, C1 to C3, U1 to U2
Connections:
- net y2 renamed d0
- net y3 renamed d1
- net y4 renamed d2
- net y5 renamed d3
- net y6 renamed d4
- net y7 renamed d5
- net y8 renamed d6
- net y9 renamed d7
- C3 pad 1: +3V3 -> +3V0
- C4 pad 1: +3V3 -> Net-(J1-Pin_15)
- C5 pad 1: +2V8 -> +3V0
- C6 pad 1: +2V8 -> +3V0
- C7 pad 1: +1V8 -> +3V0
- C8 pad 1: +2V8 -> +3V0
- J1 pad 1: +2V8 -> +3V0
- J1 pad 14: +1V8 -> +3V0
- J1 pad 21: +2V8 -> +3V0
- L1 pad 2: +3V3 -> +3V0
- U1 pad 5: +3V3 -> Net-(U1-VOUT)
- U2 pad 13: usb_dn -> unconnected-(U2-GPIO13/USB_D--Pad13)
- U2 pad 14: usb_dp -> unconnected-(U2-GPIO14/USB_D+-Pad14)
- U2 pad 15: unconnected-(U1-GPIO28-Pad15) -> led
- U2 pad 16: unconnected-(U1-GPIO5-Pad16) -> sd_clk
- U2 pad 17: unconnected-(U1-GPIO4-Pad17) -> sd_cd
- U2 pad 18: uart2_tx -> uart1_tx
- U2 pad 19: unconnected-(U1-GPIO15-Pad19) -> record
- U2 pad 2: +3V3 -> +3V0
- U2 pad 21: unconnected-(U1-GPIO23-Pad21) -> sd_cmd
- U2 pad 23: unconnected-(U1-GPIO24-Pad23) -> sd_data
- U2 pad 3: mcu_rst -> unconnected-(U2-EN/CHIP_PU-Pad3)
Other:
- board size 19.7 x 22.9 mm -> 19.1 x 21.8 mm
- board text added: "C5-Air"
- board text added: "OV5640"

Commit message: Add files via upload
Parts:
- added J9: Conn_01x01_Pin, Library:SolderWirePad_1x01_SMD_2x3mm, F.Cu at (157.2, 80.5)
- SW1: value SW_Push -> record
- moved C8 16.6 mm to (157.4, 82.5), turned to 180 degrees
- moved J4 15.7 mm to (157.1, 75.3)
- moved J5 15.5 mm to (141.7, 80.5)
- moved J6 15.4 mm to (141.7, 77.9)
- moved J7 2.58 mm to (157.1, 77.9)
- moved R6 1.51 mm to (141.4, 82.5), turned to 180 degrees
Connections:
- J1 pad 1: +3V0 -> unconnected-(J1-Pin_1-Pad1)
- J1 pad 2: GND -> unconnected-(J1-Pin_2-Pad2)
- U2 pad 13: unconnected-(U2-GPIO13/USB_D--Pad13) -> uart1_rx
- U2 pad 14: unconnected-(U2-GPIO14/USB_D+-Pad14) -> uart1_tx
- U2 pad 18: uart1_tx -> unconnected-(U2-GPIO27-Pad18)
Other:
- board text added: "to do: custom footprint for the switch (smaller courtyard) custom footprint for the esp32 (shorter pins) other sd card connector (no sd detection needed) verify if the camera connector would fit custom footprint for the inductor (longer pins)"
Changed lines of the file:
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@@
 			)
 		)
-		(property "Value" "SW_Push"
+		(property "Value" "record"
 			(at 0 2.5 0)
 			(layer "F.Fab")
@@
 	(footprint "Resistor_SMD:R_0603_1608Metric"
 		(layer "F.Cu")
-		(at 142.41 81.38 -90)
+		(at 141.36 82.47 180)
 		(descr "Resistor SMD 0603 (1608 Metric), square (rectangular) end terminal, IPC-7351 nominal, (Body size source: IPC-SM-782 page 72, https://www.pcb-3d.com/wordpress/wp-content/uploads/ipc-sm-782a_amendment_1_and_2.pdf)")
 		(tags "resistor")
 		(property "Reference" "R6"
-			(at 0 -1.43 90)
+			(at 0 -1.43 0)
 			(layer "F.SilkS")
 			(hide yes)
@@
 		)
 		(property "Value" "100kR"
-			(at 0 1.43 90)
+			(at 0 1.43 0)
 			(layer "F.Fab")
 			(effects
@@
 		)
 		(property "Datasheet" ""
-			(at 0 0 90)
+			(at 0 0 0)
 			(layer "F.Fab")
 			(hide yes)
@@
 		)
 		(property "Description" ""
-			(at 0 0 90)
+			(at 0 0 0)
 			(layer "F.Fab")
 			(hide yes)
@@
 		)
 		(property "KiLib_Generator" "SMD_2terminal_chip_molded"
-			(at 0 0 90)
+			(at 0 0 0)
 			(layer "F.SilkS")
 			(hide yes)
@@
 		)
 		(fp_text user "${REFERENCE}"
-			(at 0 0 90)
+			(at 0 0 0)
 			(layer "F.Fab")
 			(effects
@@
 		)
 		(pad "1" smd roundrect
-			(at -0.825 0 270)
+			(at -0.825 0 180)
 			(size 0.8 0.95)
 			(layers "F.Cu" "F.Mask" "F.Paste")
@@
 		)
 		(pad "2" smd roundrect
-			(at 0.825 0 270)
+			(at 0.825 0 180)
 			(size 0.8 0.95)
 			(layers "F.Cu" "F.Mask" "F.Paste")
@@
 	(footprint "Capacitor_SMD:C_0603_1608Metric"
 		(layer "F.Cu")
-		(at 140.81 81.38 90)
+		(at 157.42 82.5 180)
 		(descr "Capacitor SMD 0603 (1608 Metric), square (rectangular) end terminal, IPC-7351 nominal, (Body size source: IPC-SM-782 page 76, https://www.pcb-3d.com/wordpress/wp-content/uploads/ipc-sm-782a_amendment_1_and_2.pdf)")
 		(tags "capacitor")
 		(property "Reference" "C8"
-			(at 0 -1.43 90)
+			(at 0 -1.43 0)
 			(layer "F.SilkS")
 			(hide yes)
@@
 		)
 		(property "Value" "10uF"
-			(at 0 1.43 90)
+			(at 0 1.43 0)
 			(layer "F.Fab")
 			(effects
@@
 		)
 		(property "Datasheet" ""
-			(at 0 0 90)
+			(at 0 0 0)
 			(layer "F.Fab")
 			(hide yes)
@@
 		)
 		(property "Description" ""
-			(at 0 0 90)
+			(at 0 0 0)
 			(layer "F.Fab")
 			(hide yes)
@@
 		)
 		(property "KiLib_Generator" "SMD_2terminal_chip_molded"
-			(at 0 0 90)
+			(at 0 0 0)
 			(layer "F.SilkS")
 			(hide yes)
@@
 		(duplicate_pad_numbers_are_jumpers no)
 		(fp_line
-			(start -0.14058 -0.51)
-			(end 0.14058 -0.51)
+			(start -0.14058 0.51)
+			(end 0.14058 0.51)
 			(stroke
 				(width 0.12)
@@
 		)
 		(fp_line
-			(start -0.14058 0.51)
-			(end 0.14058 0.51)
+			(start -0.14058 -0.51)
+			(end 0.14058 -0.51)
 			(stroke
 				(width 0.12)
@@
 		)
 		(fp_text user "${REFERENCE}"
-			(at 0 0 90)
+			(at 0 0 0)
 			(layer "F.Fab")
 			(effects
@@
 		)
 		(pad "1" smd roundrect
-			(at -0.775 0 90)
+			(at -0.775 0 180)
 			(size 0.9 0.95)
 			(layers "F.Cu" "F.Mask" "F.Paste")
@@
 		)
 		(pad "2" smd roundrect
-			(at 0.775 0 90)
+			(at 0.775 0 180)
 			(size 0.9 0.95)
 			(layers "F.Cu" "F.Mask" "F.Paste")
@@
 	(footprint "Library:SolderWirePad_1x01_SMD_2x3mm"
 		(layer "F.Cu")
-		(at 157.13 81.61 90)
+		(at 141.7 80.49 90)
 		(descr "Wire Pad, Square, SMD Pad,  2mm x 4mm")
 		(tags "MeasurementPoint Square SMDPad 2mmx4mm ")
@@
 	(footprint "Library:SolderWirePad_1x01_SMD_2x3mm"
 		(layer "F.Cu")
-		(at 141.69 78.36 90)
+		(at 157.13 75.26 90)
 		(descr "Wire Pad, Square, SMD Pad,  2mm x 4mm")
 		(tags "MeasurementPoint Square SMDPad 2mmx4mm ")
@@
 			(size 0.3 1.1)
 			(layers "F.Cu" "F.Mask" "F.Paste")
-			(net "+3V0")
+			(net "unconnected-(J1-Pin_1-Pad1)")
 			(pinfunction "Pin_1_1")
-			(pintype "passive")
+			(pintype "passive+no_connect")
 		)
 		(pad "2" smd rect
@@
 			(size 0.3 1.1)
 			(layers "F.Cu" "F.Mask" "F.Paste")
-			(net "GND")
+			(net "unconnected-(J1-Pin_2-Pad2)")
 			(pinfunction "Pin_2_2")
-			(pintype "passive")
+			(pintype "passive+no_connect")
 		)
 		(pad "3" smd rect
@@
 	(footprint "Library:SolderWirePad_1x01_SMD_2x3mm"
 		(layer "F.Cu")
-		(at 157.13 75.29 90)
+		(at 157.13 77.87 90)
 		(descr "Wire Pad, Square, SMD Pad,  2mm x 4mm")
 		(tags "MeasurementPoint Square SMDPad 2mmx4mm ")
@@
 	(footprint "Library:SolderWirePad_1x01_SMD_2x3mm"
 		(layer "F.Cu")
-		(at 157.13 78.36 90)
+		(at 141.69 77.89 90)
 		(descr "Wire Pad, Square, SMD Pad,  2mm x 4mm")
 		(tags "MeasurementPoint Square SMDPad 2mmx4mm ")
@@
 		)
 	)
+	(footprint "Library:SolderWirePad_1x01_SMD_2x3mm"
+		(layer "F.Cu")
+		(at 157.16 80.49 90)
+		(descr "Wire Pad, Square, SMD Pad,  2mm x 4mm")
+		(tags "MeasurementPoint Square SMDPad 2mmx4mm ")
+		(property "Reference" "J9"
+			(at 0 -2.45 90)
+			(layer "F.SilkS")
+			(hide yes)
+			(effects
+				(font
+					(size 1 1)
+					(thickness 0.15)
+				)
+			)
+		)
+		(property "Value" "Conn_01x01_Pin"
+			(at 0 2.54 90)
+			(layer "F.Fab")
+			(effects
+				(font
+					(size 1 1)
+					(thickness 0.15)
+				)
+			)
+		)
+		(property "Datasheet" ""
+			(at 0 0 90)
+			(layer "F.Fab")
+			(hide yes)
+			(effects
+				(font
+					(size 1.27 1.27)
+					(thickness 0.15)
+				)
+			)
+		)
+		(property "Description" ""
+			(at 0 0 90)
+			(layer "F.Fab")
+			(hide yes)
+			(effects
+				(font
+					(size 1.27 1.27)
+					(thickness 0.15)
+				)
+			)
+		)
+		(property ki_fp_filters "Connector*:*_1x??_*")
+		(sheetname "/")
+		(sheetfile "esp32c5-airunit-nano.kicad_sch")
+		(units
+			(unit
+				(name "A")
+				(pins "1")
+			)
+		)
+		(duplicate_pad_numbers_are_jumpers no)
+		(fp_rect
+			(start -1.25 -1.75)
+			(end 1.25 1.75)
+			(stroke
+				(width 0.05)
+				(type solid)
+			)
+			(fill no)
+			(layer "F.CrtYd")
+		)
+		(fp_rect
+			(start -1.15 -1.643638)
+			(end 1.15 1.644324)
+			(stroke
+				(width 0.1)
+				(type default)
+			)
+			(fill no)
+			(layer "F.Fab")
+		)
+		(fp_text user "${REFERENCE}"
+			(at 0 0 90)
+			(layer "F.Fab")
+			(effects
+				(font
+					(size 1 1)
+					(thickness 0.15)
+				)
+			)
+		)
+		(pad "1" smd roundrect
+			(at 0 0 90)
+			(size 2 3)
+			(layers "F.Cu" "F.Mask")
+			(roundrect_rratio 0.25)
+			(net "uart1_rx")
+			(pinfunction "Pin_1_1")
+			(pintype "passive")
+		)
+		(embedded_fonts no)
+	)
 	(footprint "Capacitor_SMD:C_0603_1608Metric"
 		(layer "F.Cu")
@@
 			(size 1.5 0.9)
 			(layers "B.Cu" "B.Mask" "B.Paste")
-			(net "unconnected-(U2-GPIO13{slash}USB_D--Pad13)")
+			(net "uart1_rx")
 			(pinfunction "GPIO13/USB_D-_13")
-			(pintype "bidirectional+no_connect")
+			(pintype "bidirectional")
 		)
 		(pad "14" smd rect
@@
 			(size 1.5 0.9)
 			(layers "B.Cu" "B.Mask" "B.Paste")
-			(net "unconnected-(U2-GPIO14{slash}USB_D+-Pad14)")
+			(net "uart1_tx")
 			(pinfunction "GPIO14/USB_D+_14")
-			(pintype "bidirectional+no_connect")
+			(pintype "bidirectional")
 		)
 		(pad "15" smd rect
@@
 			(size 1.5 0.9)
 			(layers "B.Cu" "B.Mask" "B.Paste")
-			(net "uart1_tx")
+			(net "unconnected-(U2-GPIO27-Pad18)")
 			(pinfunction "GPIO27_18")
-			(pintype "bidirectional")
+			(pintype "bidirectional+no_connect")
 		)
 		(pad "19" smd rect
@@
 		)
 	)
+	(gr_text "to do:\ncustom footprint for the switch (smaller courtyard)\ncustom footprint for the esp32 (shorter pins)\nother sd card connector (no sd detection needed)\nverify if the camera connector would fit\ncustom footprint for the inductor (longer pins)"
+		(at 129.82 65.34 0)
+		(layer "F.SilkS")
+		(effects
+			(font
+				(size 1.5 1.5)
+				(thickness 0.3)
+				(bold yes)
+			)
+			(justify left bottom)
+		)
+	)
