File: project/esp32c5-airunit-nano.kicad_sch (KiCad schematic)
At the start: 26 parts, among them J1 FPC0.5B-WTX-24P, J2 Conn_01x01_Pin, J4 Conn_01x01_Pin, J5 Conn_01x01_Pin, J6 Conn_01x01_Pin, J7 Conn_01x01_Pin, J8 0475710001, J9 Conn_01x01_Pin, SW1 record, U1 MT3406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

Commit message: i've updated the schematic and changed the button for a cheaper one
Parts:
- C1, C6: value 100nF -> 100nF 10V
- C2, C3, C4, C5, C7, C8: value 10uF -> 10uF 10V
- D1: value red -> NCD0603R2
- J8: value 0475710001 -> TF-021B-H265
- R2: value tbd -> 22kR
- SW1: value record -> EVQP7C01P; footprint Button_Switch_SMD:SW_SPST_B3U-3000P-B -> Button_Switch_SMD:SW_SPST_EVQP7C
- U2: value ESP32-C5-WROOM-1U -> ESP32-C5-WROOM-1U-N8R8
Other:
- note added: "all passive elements (resistors, capacitors) are in 0603 package"
Changed lines of the file:
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@@
 	(title_block
 		(title "esp32c5-airunit-nano")
-		(date "2026-05-30")
+		(date "2026-06-05")
+		(rev "V1.0")
 		(company "us3r_d0e5nt_3x1st")
 	)
@@
 		)
 	)
+	(text "all passive elements (resistors, capacitors) are in 0603 package"
+		(exclude_from_sim no)
+		(at 62.992 64.516 0)
+		(effects
+			(font
+				(size 1.27 1.27)
+			)
+		)
+	)
 	(text "vddaf\ngnd\ny4\ny3\ny5\ny2\ny6\npclk\ny7\ngnd\ny8\nmclk\ny9\nvdddo\nvddd\nhsync\npwdn\nvsync\nrst\nscl\nvdda\nsda\ngnd\nstrobe"
 		(exclude_from_sim no)
@@
 		)
 		(property "Value" "100kR"
-			(at 73.914 47.752 90)
+			(at 72.898 47.752 90)
 			(show_name no)
 			(do_not_autoplace no)
@@
 			)
 		)
-		(property "Value" "10uF"
-			(at 83.058 53.594 0)
+		(property "Value" "10uF 10V"
+			(at 77.47 53.594 0)
 			(show_name no)
 			(do_not_autoplace no)
@@
 			)
 		)
-		(property "Value" "red"
+		(property "Value" "NCD0603R2"
 			(at 37.338 171.196 90)
 			(show_name no)
@@
 			)
 		)
-		(property "Value" "10uF"
+		(property "Value" "10uF 10V"
 			(at 187.198 110.744 0)
 			(show_name no)
@@
 			)
 		)
-		(property "Value" "tbd"
+		(property "Value" "22kR"
 			(at 70.866 54.102 0)
 			(show_name no)
@@
 			)
 		)
-		(property "Value" "10uF"
-			(at 243.84 83.058 90)
+		(property "Value" "10uF 10V"
+			(at 247.65 83.312 90)
 			(show_name no)
 			(do_not_autoplace no)
@@
 			)
 		)
-		(property "Value" "10uF"
-			(at 43.688 53.848 0)
+		(property "Value" "10uF 10V"
+			(at 38.1 53.848 0)
 			(show_name no)
 			(do_not_autoplace no)
@@
 	)
 	(symbol
+		(lib_id "Switch:SW_Push")
+		(at 66.04 165.1 90)
+		(unit 1)
+		(body_style 1)
+		(exclude_from_sim no)
+		(in_bom yes)
+		(on_board yes)
+		(in_pos_files yes)
+		(dnp no)
+		(fields_autoplaced yes)
+		(property "Reference" "SW1"
+			(at 67.31 163.8299 90)
+			(show_name no)
+			(do_not_autoplace no)
+			(effects
+				(font
+					(size 1.27 1.27)
+				)
+				(justify right)
+			)
+		)
+		(property "Value" "EVQP7C01P"
+			(at 67.31 166.3699 90)
+			(show_name no)
+			(do_not_autoplace no)
+			(effects
+				(font
+					(size 1.27 1.27)
+				)
+				(justify right)
+			)
+		)
+		(property "Footprint" "Button_Switch_SMD:SW_SPST_EVQP7C"
+			(at 60.96 165.1 0)
+			(hide yes)
+			(show_name no)
+			(do_not_autoplace no)
+			(effects
+				(font
+					(size 1.27 1.27)
+				)
+			)
+		)
+		(property "Datasheet" ""
+			(at 60.96 165.1 0)
+			(hide yes)
+			(show_name no)
+			(do_not_autoplace no)
+			(effects
+				(font
+					(size 1.27 1.27)
+				)
+			)
+		)
+		(property "Description" "Push button switch, generic, two pins"
+			(at 66.04 165.1 0)
+			(hide yes)
+			(show_name no)
+			(do_not_autoplace no)
+			(effects
+				(font
+					(size 1.27 1.27)
+				)
+			)
+		)
+		(pin "2"
+		)
+		(pin "1"
+		)
+		(instances
+			(project "esp32c5-airunit-nano"
+				(path "/d536f07d-edbd-473f-b507-96822d187be1"
+					(reference "SW1")
+					(unit 1)
+				)
+			)
+		)
+	)
+	(symbol
 		(lib_id "power:GND")
 		(at 242.57 80.01 90)
@@
 			)
 		)
-		(property "Value" "100nF"
-			(at 30.48 53.848 0)
+		(property "Value" "100nF 10V"
+			(at 25.908 54.102 0)
 			(show_name no)
 			(do_not_autoplace no)
@@
 			)
 		)
-		(property "Value" "10uF"
-			(at 246.634 100.838 0)
+		(property "Value" "10uF 10V"
+			(at 246.888 100.838 0)
 			(show_name no)
 			(do_not_autoplace no)
@@
 			)
 		)
-		(property "Value" "10uF"
-			(at 144.78 53.594 0)
+		(property "Value" "10uF 10V"
+			(at 140.208 53.594 0)
 			(show_name no)
 			(do_not_autoplace no)
@@
 		(dnp no)
 		(property "Reference" "U2"
-			(at 78.994 77.978 0)
+			(at 73.914 78.232 0)
 			(show_name no)
 			(do_not_autoplace no)
@@
 			)
 		)
-		(property "Value" "ESP32-C5-WROOM-1U"
-			(at 78.994 80.518 0)
+		(property "Value" "ESP32-C5-WROOM-1U-N8R8"
+			(at 73.914 80.772 0)
 			(show_name no)
 			(do_not_autoplace no)
@@
 			)
 		)
-		(property "Value" "0475710001"
+		(property "Value" "TF-021B-H265"
 			(at 165.1 96.52 0)
 			(show_name no)
@@
 	)
 	(symbol
-		(lib_id "Switch:SW_Push")
-		(at 66.04 165.1 90)
-		(unit 1)
-		(body_style 1)
-		(exclude_from_sim no)
-		(in_bom yes)
-		(on_board yes)
-		(in_pos_files yes)
-		(dnp no)
-		(fields_autoplaced yes)
-		(property "Reference" "SW1"
-			(at 67.31 163.8299 90)
-			(show_name no)
-			(do_not_autoplace no)
-			(effects
-				(font
-					(size 1.27 1.27)
-				)
-				(justify right)
-			)
-		)
-		(property "Value" "record"
-			(at 67.31 166.3699 90)
-			(show_name no)
-			(do_not_autoplace no)
-			(effects
-				(font
-					(size 1.27 1.27)
-				)
-				(justify right)
-			)
-		)
-		(property "Footprint" "Button_Switch_SMD:SW_SPST_B3U-3000P-B"
-			(at 60.96 165.1 0)
-			(hide yes)
-			(show_name no)
-			(do_not_autoplace no)
-			(effects
-				(font
-					(size 1.27 1.27)
-				)
-			)
-		)
-		(property "Datasheet" ""
-			(at 60.96 165.1 0)
-			(hide yes)
-			(show_name no)
-			(do_not_autoplace no)
-			(effects
-				(font
-					(size 1.27 1.27)
-				)
-			)
-		)
-		(property "Description" "Push button switch, generic, two pins"
-			(at 66.04 165.1 0)
-			(hide yes)
-			(show_name no)
-			(do_not_autoplace no)
-			(effects
-				(font
-					(size 1.27 1.27)
-				)
-			)
-		)
-		(pin "1"
-		)
-		(pin "2"
-		)
-		(instances
-			(project "esp32c5-airunit-nano"
-				(path "/d536f07d-edbd-473f-b507-96822d187be1"
-					(reference "SW1")
-					(unit 1)
-				)
-			)
-		)
-	)
-	(symbol
 		(lib_id "power:VCC")
 		(at 36.83 40.64 0)
@@
 			)
 		)
-		(property "Value" "100nF"
+		(property "Value" "100nF 10V"
 			(at 89.408 53.594 0)
 			(show_name no)

Commit message: the R2 should be 25kR
Parts:
- R2: value 22kR -> 25kR
Changed lines of the file:
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@@
 			)
 		)
-		(property "Value" "22kR"
+		(property "Value" "25kR"
 			(at 70.866 54.102 0)
 			(show_name no)

Commit message: Add files via upload
Connections:
- net +3V0: now also Y1.1 (Tri-State)
- no-connect marks 13 -> 12
Changed lines of the file:
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@@
+	)
+	(junction
+		(at 153.67 44.45)
+		(diameter 0)
+		(color 0 0 0 0)
 	)
 	(junction
@@
 	)
 	(no_connect
-		(at 153.67 53.34)
-	)
-	(no_connect
 		(at 237.49 44.45)
 	)
@@
 	(wire
 		(pts
+			(xy 153.67 44.45) (xy 153.67 53.34)
+		)
+		(stroke
+			(width 0)
+			(type default)
+		)
+	)
+	(wire
+		(pts
 			(xy 135.89 170.18) (xy 134.62 170.18)
 		)
@@
 	(wire
 		(pts
+			(xy 153.67 44.45) (xy 163.83 44.45)
+		)
+		(stroke
+			(width 0)
+			(type default)
+		)
+	)
+	(wire
+		(pts
 			(xy 66.04 171.45) (xy 66.04 170.18)
 		)
@@
 	(wire
 		(pts
-			(xy 149.86 44.45) (xy 163.83 44.45)
-		)
-		(stroke
+			(xy 149.86 44.45) (xy 153.67 44.45)
+		)
+		(stroke

Commit message: i've updated the files
there were some major errors in the v1.0 of the project
Parts:
- R1, R6: value 100kR -> 47kR
- R2: value 25kR -> 12kR
Connections:
- net +3V0: now also U2.3 (EN/CHIP_PU)
- net GND: now also J1.17 (Pin_17)
- net d0: now also U2.9 (GPIO7); no longer U2.11 (GPIO9)
- net d1: now also U2.11 (GPIO9); no longer U2.13 (GPIO13/USB_D-)
- net d2: now also U2.12 (GPIO10); no longer U2.14 (GPIO14/USB_D+)
- net d3: now also U2.10 (GPIO8); no longer U2.12 (GPIO10)
- net d4: now also U2.8 (GPIO6); no longer U2.10 (GPIO8)
- net d5: now also U2.6 (GPIO0); no longer U2.8 (GPIO6)
- net d6: now also U2.5 (GPIO3); no longer U2.7 (GPIO1)
- net d7: now also U2.4 (GPIO2); no longer U2.17 (GPIO4)
- net led: now also U2.18 (GPIO27); no longer U2.4 (GPIO2)
- net pclk: now also U2.7 (GPIO1); no longer U2.9 (GPIO7)
- net record: now also U2.15 (GPIO28); no longer U2.27 (GPIO26)
- net scl: now also U2.17 (GPIO4); no longer U2.16 (GPIO5)
- net sd_cd: now also U2.21 (GPIO23); no longer U2.19 (GPIO15)
- net sd_clk: now also U2.26 (GPIO25); no longer U2.21 (GPIO23)
- net sd_cmd: now also U2.23 (GPIO24); no longer U2.18 (GPIO27)
- net sd_data: now also U2.27 (GPIO26); no longer U2.23 (GPIO24)
- net sda: now also U2.16 (GPIO5); no longer U2.15 (GPIO28)
- net uart1_rx: now also U2.13 (GPIO13/USB_D-); no longer U2.6 (GPIO0)
- net uart1_tx: now also U2.14 (GPIO14/USB_D+); no longer U2.5 (GPIO3)
- no-connect marks 12 -> 10
Other:
- note added: "bootloader: GPIO28 to GND"
- note removed: "reset the mcu: EN to GND bootloader: GPIO28 to GND"

Commit message: i've uploaded the v1.2
Parts:
- removed C7: 10uF 10V, Capacitor_SMD:C_0603_1608Metric, symbol Device:C
- removed Y1: YD24MUBCE2O, Oscillator:Oscillator_SMD_ECS_2520MV-xxx-xx-4Pin_2.5x2.0mm, symbol Oscillator:ECS-2520MV-xxx-xx
Connections:
- net record: now also D1.1 (K)
- net xclk: now also U2.18 (GPIO27)
- removed net led: D1.1 (K), U2.18 (GPIO27)
Other:
- moved on the sheet: C4, C5, C8, D1, J1, J8, R3, R6, SW1
